Commit message: better sim

File: urdf/bebop2.urdf (robot description, URDF)
Before this commit: robot bebop2, 5 links, 4 joints
Links:
- removed link base_link
- added link base_link_ekf; visual mesh filename=package://nero_drone/meshes/bebop.dae scale=0.001 0.001 0.001
Joints:
- joint joint_propeller_back_left: parent base_link -> base_link_ekf
- joint joint_propeller_back_right: parent base_link -> base_link_ekf
- joint joint_propeller_front_left: parent base_link -> base_link_ekf
- joint joint_propeller_front_right: parent base_link -> base_link_ekf

Commit message: Refactor: rename package to neroControl and update README dependencies

File: urdf/bebop2.urdf (robot description, URDF)
Before this commit: robot bebop2, 5 links, 4 joints
Links:
- link base_link_ekf: geometry visual mesh filename=package://neroControl/meshes/bebop.dae scale=0.001 0.001 0.001
- link propeller_back_left: geometry visual mesh filename=package://neroControl/meshes/propeller_cw.dae scale=0.0007 0.0007 0.0007
- link propeller_back_right: geometry visual mesh filename=package://neroControl/meshes/propeller_ccw.dae scale=0.0007 0.0007 0.0007
- link propeller_front_left: geometry visual mesh filename=package://neroControl/meshes/propeller_ccw.dae scale=0.0007 0.0007 0.0007
- link propeller_front_right: geometry visual mesh filename=package://neroControl/meshes/propeller_cw.dae scale=0.0007 0.0007 0.0007
